File: board/SID-Monitor.sch (EAGLE design)
At the start: 107 parts, among them IC1 LM317, IC2 LM337, IC3 TLE2082, IC4 TLE2082, IC5 MAX275ACP, IC6 TLE2082, IC7 TLE2082, IC8 TLE2082, IC9 PHOTON_WITH_HEADERS, J101 POWERJACK-PTH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

Commit message: Board layout first pass
Parts:
- C1002, C107, C108, C701: device SaintGimp:CAP-POL-3.5-8 -> SaintGimp:CAPACITOR-POLARIZED-3.5-8
- C101, C102: device SaintGimp:CAP-POL-5-13 -> SaintGimp:CAPACITOR-POLARIZED-5-13
- C105, C106: device SaintGimp:CAP-POL-2.5-5 -> SaintGimp:CAPACITOR-POLARIZED-2.5-5
- C401, C402: device SaintGimp:CAPACITOR-2.5MM -> SaintGimp:CAPACITOR-5MM
- D101, D102, D103, D104, D105, D106: device SaintGimp:DIODE1N4001 -> SaintGimp:DIODE-1N4001
- D601, D602: device SaintGimp:DIODE1N4148 -> SaintGimp:DIODE-1N4148
- IC9: value PHOTON_WITH_HEADERS -> PHOTON
Connections:
- new net N$39: IC8B.-IN, IC8B.OUT
- net GND: now also IC8B.+IN

Commit message: Update values to tune to 25.2 kHz
Parts:
- R101, R102: value 240 -> 270
- R309: value 51 -> 49.9
- R401, R406: value 47k -> 120k
- R402, R407: value 75k -> 360k
- R403, R408: value 30.9k -> 75k
- R404, R405: value 28.7k -> 75k
- RV401, RV402: value 5K -> 10k
- RV801: value 1K -> 1k
Connections:
- net GND: now also RV102.S
Changed lines of the file:
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@@
 <?xml version="1.0" encoding="utf-8"?>
 <!DOCTYPE eagle SYSTEM "eagle.dtd">
-<eagle version="8.4.1">
+<eagle version="8.5.1">
 <drawing>
 <settings>
@@
 <part name="JP401" library="SaintGimp" deviceset="JUMPER1" device=""/>
 <part name="IC5" library="SaintGimp" deviceset="MAX275" device="ACP"/>
-<part name="R401" library="SaintGimp" deviceset="RESISTOR-*" device="7.5MM" value="47k"/>
-<part name="R402" library="SaintGimp" deviceset="RESISTOR-*" device="7.5MM" value="75k"/>
-<part name="R403" library="SaintGimp" deviceset="RESISTOR-*" device="7.5MM" value="30.9k"/>
-<part name="R404" library="SaintGimp" deviceset="RESISTOR-*" device="7.5MM" value="28.7k"/>
-<part name="RV401" library="SaintGimp" deviceset="POT" device="TRIM" value="5K"/>
+<part name="R401" library="SaintGimp" deviceset="RESISTOR-*" device="7.5MM" value="120k"/>
+<part name="R402" library="SaintGimp" deviceset="RESISTOR-*" device="7.5MM" value="360k"/>
+<part name="R403" library="SaintGimp" deviceset="RESISTOR-*" device="7.5MM" value="75k"/>
+<part name="R404" library="SaintGimp" deviceset="RESISTOR-*" device="7.5MM" value="75k"/>
+<part name="RV401" library="SaintGimp" deviceset="POT" device="TRIM" value="10k"/>
 <part name="JP402" library="SaintGimp" deviceset="JUMPER1" device=""/>
 <part name="C405" library="SaintGimp" deviceset="CAPACITOR" device="-2.5MM" value="0.1uF"/>
-<part name="R406" library="SaintGimp" deviceset="RESISTOR-*" device="7.5MM" value="47k"/>
-<part name="R405" library="SaintGimp" deviceset="RESISTOR-*" device="7.5MM" value="28.7k"/>
-<part name="R407" library="SaintGimp" deviceset="RESISTOR-*" device="7.5MM" value="75k"/>
-<part name="R408" library="SaintGimp" deviceset="RESISTOR-*" device="7.5MM" value="30.9k"/>
-<part name="RV402" library="SaintGimp" deviceset="POT" device="TRIM" value="5K"/>
+<part name="R406" library="SaintGimp" deviceset="RESISTOR-*" device="7.5MM" value="120k"/>
+<part name="R405" library="SaintGimp" deviceset="RESISTOR-*" device="7.5MM" value="75k"/>
+<part name="R407" library="SaintGimp" deviceset="RESISTOR-*" device="7.5MM" value="360k"/>
+<part name="R408" library="SaintGimp" deviceset="RESISTOR-*" device="7.5MM" value="75k"/>
+<part name="RV402" library="SaintGimp" deviceset="POT" device="TRIM" value="10k"/>
 <part name="P-208" library="SaintGimp" deviceset="-5V" device=""/>
 <part name="P-210" library="SaintGimp" deviceset="-5V" device=""/>
@@
 <part name="X301" library="SaintGimp" deviceset="5414373" device=""/>
 <part name="GND212" library="SaintGimp" deviceset="GND" device=""/>
-<part name="R309" library="SaintGimp" deviceset="RESISTOR-*" device="7.5MM" value="51"/>
+<part name="R309" library="SaintGimp" deviceset="RESISTOR-*" device="7.5MM" value="49.9"/>
 <part name="IC6" library="SaintGimp" deviceset="TLE2082" device=""/>
 <part name="R602" library="SaintGimp" deviceset="RESISTOR-*" device="7.5MM" value="10k"/>
@@
 <part name="P+204" library="SaintGimp" deviceset="+5V" device=""/>
 <part name="R803" library="SaintGimp" deviceset="RESISTOR-*" device="7.5MM" value="47k"/>
-<part name="RV801" library="SaintGimp" deviceset="POT" device="TRIM" value="1K"/>
+<part name="RV801" library="SaintGimp" deviceset="POT" device="TRIM" value="1k"/>
 <part name="R804" library="SaintGimp" deviceset="RESISTOR-*" device="7.5MM" value="47k"/>
 <part name="P-204" library="SaintGimp" deviceset="-5V" device=""/>
@@
 <part name="RV101" library="SaintGimp" deviceset="POT" device="TRIM" value="1k"/>
 <part name="C105" library="SaintGimp" deviceset="CAPACITOR-POLARIZED" device="-2.5-5" value="10uf"/>
-<part name="R101" library="SaintGimp" deviceset="RESISTOR-*" device="7.5MM" value="240"/>
+<part name="R101" library="SaintGimp" deviceset="RESISTOR-*" device="7.5MM" value="270"/>
 <part name="RV102" library="SaintGimp" deviceset="POT" device="TRIM" value="1k"/>
 <part name="C106" library="SaintGimp" deviceset="CAPACITOR-POLARIZED" device="-2.5-5" value="10uf"/>
-<part name="R102" library="SaintGimp" deviceset="RESISTOR-*" device="7.5MM" value="240"/>
+<part name="R102" library="SaintGimp" deviceset="RESISTOR-*" device="7.5MM" value="270"/>
 <part name="GND1" library="SaintGimp" deviceset="GND" device=""/>
 </parts>
@@
 <pinref part="C106" gate="G$1" pin="+"/>
 <wire x1="58.42" y1="48.26" x2="58.42" y2="50.8" width="0.1524" layer="91"/>
+<pinref part="RV102" gate="G$1" pin="S"/>
+<wire x1="48.26" y1="43.18" x2="48.26" y2="50.8" width="0.1524" layer="91"/>
 </segment>
 <segment>
